Commit message: URDF_update

File: nanny_description/urdf/nanny.xacro (robot description, xacro)
@@ -19,5 +19,5 @@
   </inertial>
   <visual>
-    <origin rpy="0 0 0" xyz="0 0 0"/>
+    <origin rpy="0 0 0" xyz="0 0 0.021978"/>
     <geometry>
       <mesh filename="package://nanny_description/meshes/base_link.stl" scale="0.001 0.001 0.001"/>
@@ -26,5 +26,5 @@
   </visual>
   <collision>
-    <origin rpy="0 0 0" xyz="0 0 0"/>
+    <origin rpy="0 0 0" xyz="0 0 0.021978"/>
     <geometry>
       <mesh filename="package://nanny_description/meshes/base_link.stl" scale="0.001 0.001 0.001"/>
@@ -39,5 +39,5 @@
   </inertial>
   <visual>
-    <origin rpy="0 0 0" xyz="-0.144318 0.27111 -0.011978"/>
+    <origin rpy="0 0 0" xyz="-0.144318 0.27111 0.01"/>
     <geometry>
       <mesh filename="package://nanny_description/meshes/motor_v1__1__1.stl" scale="0.001 0.001 0.001"/>
@@ -46,5 +46,5 @@
   </visual>
   <collision>
-    <origin rpy="0 0 0" xyz="-0.144318 0.27111 -0.011978"/>
+    <origin rpy="0 0 0" xyz="-0.144318 0.27111 0.01"/>
     <geometry>
       <mesh filename="package://nanny_description/meshes/motor_v1__1__1.stl" scale="0.001 0.001 0.001"/>
@@ -59,5 +59,5 @@
   </inertial>
   <visual>
-    <origin rpy="0 0 0" xyz="-0.808518 0.27111 -0.011978"/>
+    <origin rpy="0 0 0" xyz="-0.808518 0.27111 0.01"/>
     <geometry>
       <mesh filename="package://nanny_description/meshes/motor_v1_1.stl" scale="0.001 0.001 0.001"/>
@@ -66,5 +66,5 @@
   </visual>
   <collision>
-    <origin rpy="0 0 0" xyz="-0.808518 0.27111 -0.011978"/>
+    <origin rpy="0 0 0" xyz="-0.808518 0.27111 0.01"/>
     <geometry>
       <mesh filename="package://nanny_description/meshes/motor_v1_1.stl" scale="0.001 0.001 0.001"/>
@@ -79,5 +79,5 @@
   </inertial>
   <visual>
-    <origin rpy="0 0 0" xyz="-0.068818 0.271212 -0.056647"/>
+    <origin rpy="0 0 0" xyz="-0.068818 0.271212 -0.034669"/>
     <geometry>
       <mesh filename="package://nanny_description/meshes/wheel_v1__1__1.stl" scale="0.001 0.001 0.001"/>
@@ -86,5 +86,5 @@
   </visual>
   <collision>
-    <origin rpy="0 0 0" xyz="-0.068818 0.271212 -0.056647"/>
+    <origin rpy="0 0 0" xyz="-0.068818 0.271212 -0.034669"/>
     <geometry>
       <mesh filename="package://nanny_description/meshes/wheel_v1__1__1.stl" scale="0.001 0.001 0.001"/>
@@ -99,5 +99,5 @@
   </inertial>
   <visual>
-    <origin rpy="0 0 0" xyz="-0.931018 0.271009 -0.056647"/>
+    <origin rpy="0 0 0" xyz="-0.931018 0.271009 -0.034669"/>
     <geometry>
       <mesh filename="package://nanny_description/meshes/wheel_v1_1.stl" scale="0.001 0.001 0.001"/>
@@ -106,5 +106,5 @@
   </visual>
   <collision>
-    <origin rpy="0 0 0" xyz="-0.931018 0.271009 -0.056647"/>
+    <origin rpy="0 0 0" xyz="-0.931018 0.271009 -0.034669"/>
     <geometry>
       <mesh filename="package://nanny_description/meshes/wheel_v1_1.stl" scale="0.001 0.001 0.001"/>
@@ -119,5 +119,5 @@
   </inertial>
   <visual>
-    <origin rpy="0 0 0" xyz="-0.826018 0.094334 0.000722"/>
+    <origin rpy="0 0 0" xyz="-0.826018 0.094334 0.0227"/>
     <geometry>
       <mesh filename="package://nanny_description/meshes/extrude_1.stl" scale="0.001 0.001 0.001"/>
@@ -126,5 +126,5 @@
   </visual>
   <collision>
-    <origin rpy="0 0 0" xyz="-0.826018 0.094334 0.000722"/>
+    <origin rpy="0 0 0" xyz="-0.826018 0.094334 0.01"/>
     <geometry>
       <mesh filename="package://nanny_description/meshes/extrude_1.stl" scale="0.001 0.001 0.001"/>
@@ -139,5 +139,5 @@
   </inertial>
   <visual>
-    <origin rpy="0 0 0" xyz="-0.180818 0.074834 -0.011978"/>
+    <origin rpy="0 0 0" xyz="-0.180818 0.074834 0.01"/>
     <geometry>
       <mesh filename="package://nanny_description/meshes/extrude_2.stl" scale="0.001 0.001 0.001"/>
@@ -146,5 +146,5 @@
   </visual>
   <collision>
-    <origin rpy="0 0 0" xyz="-0.180818 0.074834 -0.011978"/>
+    <origin rpy="0 0 0" xyz="-0.180818 0.074834 0.01"/>
     <geometry>
       <mesh filename="package://nanny_description/meshes/extrude_2.stl" scale="0.001 0.001 0.001"/>
@@ -159,5 +159,5 @@
   </inertial>
   <visual>
-    <origin rpy="0 0 0" xyz="-0.321318 0.379834 -0.011978"/>
+    <origin rpy="0 0 0" xyz="-0.321318 0.379834 0.01"/>
     <geometry>
       <mesh filename="package://nanny_description/meshes/extrude_3.stl" scale="0.001 0.001 0.001"/>
@@ -166,5 +166,5 @@
   </visual>
   <collision>
-    <origin rpy="0 0 0" xyz="-0.321318 0.379834 -0.011978"/>
+    <origin rpy="0 0 0" xyz="-0.321318 0.379834 0.01"/>
     <geometry>
       <mesh filename="package://nanny_description/meshes/extrude_3.stl" scale="0.001 0.001 0.001"/>
@@ -179,5 +179,5 @@
   </inertial>
   <visual>
-    <origin rpy="0 0 0" xyz="-0.690018 0.369334 -0.011978"/>
+    <origin rpy="0 0 0" xyz="-0.690018 0.369334 0.01"/>
     <geometry>
       <mesh filename="package://nanny_description/meshes/extrude_4.stl" scale="0.001 0.001 0.001"/>
@@ -186,5 +186,5 @@
   </visual>
   <collision>
-    <origin rpy="0 0 0" xyz="-0.690018 0.369334 -0.011978"/>
+    <origin rpy="0 0 0" xyz="-0.690018 0.369334 0.01"/>
     <geometry>
       <mesh filename="package://nanny_description/meshes/extrude_4.stl" scale="0.001 0.001 0.001"/>
@@ -199,5 +199,5 @@
   </inertial>
   <visual>
-    <origin rpy="0 0 0" xyz="-0.519747 -0.230753 -0.011978"/>
+    <origin rpy="0 0 0" xyz="-0.519747 -0.230753 0.01"/>
     <geometry>
       <mesh filename="package://nanny_description/meshes/extrude_5.stl" scale="0.001 0.001 0.001"/>
@@ -206,5 +206,5 @@
   </visual>
   <collision>
-    <origin rpy="0 0 0" xyz="-0.519747 -0.230753 -0.011978"/>
+    <origin rpy="0 0 0" xyz="-0.519747 -0.230753 0.01"/>
     <geometry>
       <mesh filename="package://nanny_description/meshes/extrude_5.stl" scale="0.001 0.001 0.001"/>
@@ -219,5 +219,5 @@
   </inertial>
   <visual>
-    <origin rpy="0 0 0" xyz="-0.674918 0.31791 -0.011978"/>
+    <origin rpy="0 0 0" xyz="-0.674918 0.31791 0.01"/>
     <geometry>
       <mesh filename="package://nanny_description/meshes/battery_v1_1.stl" scale="0.001 0.001 0.001"/>
@@ -226,5 +226,5 @@
   </visual>
   <collision>
-    <origin rpy="0 0 0" xyz="-0.674918 0.31791 -0.011978"/>
+    <origin rpy="0 0 0" xyz="-0.674918 0.31791 0.01"/>
     <geometry>
       <mesh filename="package://nanny_description/meshes/battery_v1_1.stl" scale="0.001 0.001 0.001"/>
@@ -239,5 +239,5 @@
   </inertial>
   <visual>
-    <origin rpy="0 0 0" xyz="-0.181515 0.330913 -0.011978"/>
+    <origin rpy="0 0 0" xyz="-0.181515 0.330913 0.01"/>
     <geometry>
       <mesh filename="package://nanny_description/meshes/bracket_v1_1.stl" scale="0.001 0.001 0.001"/>
@@ -246,5 +246,5 @@
   </visual>
   <collision>
-    <origin rpy="0 0 0" xyz="-0.181515 0.330913 -0.011978"/>
+    <origin rpy="0 0 0" xyz="-0.181515 0.330913 0.01"/>
     <geometry>
       <mesh filename="package://nanny_description/meshes/bracket_v1_1.stl" scale="0.001 0.001 0.001"/>
@@ -259,5 +259,5 @@
   </inertial>
   <visual>
-    <origin rpy="0 0 0" xyz="-0.818321 0.335913 -0.011978"/>
+    <origin rpy="0 0 0" xyz="-0.818321 0.335913 0.01"/>
     <geometry>
       <mesh filename="package://nanny_description/meshes/bracket_v1__1__1.stl" scale="0.001 0.001 0.001"/>
@@ -266,5 +266,5 @@
   </visual>
   <collision>
-    <origin rpy="0 0 0" xyz="-0.818321 0.335913 -0.011978"/>
+    <origin rpy="0 0 0" xyz="-0.818321 0.335913 0.01"/>
     <geometry>
       <mesh filename="package://nanny_description/meshes/bracket_v1__1__1.stl" scale="0.001 0.001 0.001"/>
@@ -279,5 +279,5 @@
   </inertial>
   <visual>
-    <origin rpy="0 0 0" xyz="-0.339208 0.371284 -0.220013"/>
+    <origin rpy="0 0 0" xyz="-0.339208 0.371284 -0.198035"/>
     <geometry>
       <mesh filename="package://nanny_description/meshes/universalplate_v1_1.stl" scale="0.001 0.001 0.001"/>
@@ -286,5 +286,5 @@
   </visual>
   <collision>
-    <origin rpy="0 0 0" xyz="-0.339208 0.371284 -0.220013"/>
+    <origin rpy="0 0 0" xyz="-0.339208 0.371284 -0.198035"/>
     <geometry>
       <mesh filename="package://nanny_description/meshes/universalplate_v1_1.stl" scale="0.001 0.001 0.001"/>
@@ -299,5 +299,5 @@
   </inertial>
   <visual>
-    <origin rpy="0 0 0" xyz="-0.240208 -0.166116 -0.220013"/>
+    <origin rpy="0 0 0" xyz="-0.240208 -0.166116 -0.198035"/>
     <geometry>
       <mesh filename="package://nanny_description/meshes/castorconnect_v1_1.stl" scale="0.001 0.001 0.001"/>
@@ -306,5 +306,5 @@
   </visual>
   <collision>
-    <origin rpy="0 0 0" xyz="-0.240208 -0.166116 -0.220013"/>
+    <origin rpy="0 0 0" xyz="-0.240208 -0.166116 -0.198035"/>
     <geometry>
       <mesh filename="package://nanny_description/meshes/castorconnect_v1_1.stl" scale="0.001 0.001 0.001"/>
@@ -319,5 +319,5 @@
   </inertial>
   <visual>
-    <origin rpy="0 0 0" xyz="-0.759408 -0.166116 -0.220013"/>
+    <origin rpy="0 0 0" xyz="-0.759408 -0.166116 -0.198035"/>
     <geometry>
       <mesh filename="package://nanny_description/meshes/castorconnect_v1__1__1.stl" scale="0.001 0.001 0.001"/>
@@ -326,5 +326,5 @@
   </visual>
   <collision>
-    <origin rpy="0 0 0" xyz="-0.759408 -0.166116 -0.220013"/>
+    <origin rpy="0 0 0" xyz="-0.759408 -0.166116 -0.198035"/>
     <geometry>
       <mesh filename="package://nanny_description/meshes/castorconnect_v1__1__1.stl" scale="0.001 0.001 0.001"/>
@@ -339,5 +339,5 @@
   </inertial>
   <visual>
-    <origin rpy="0 0 0" xyz="-0.253053 -0.228029 -0.080313"/>
+    <origin rpy="0 0 0" xyz="-0.253053 -0.228029 -0.058335"/>
     <geometry>
       <mesh filename="package://nanny_description/meshes/castor_v1_1.stl" scale="0.001 0.001 0.001"/>
@@ -346,5 +346,5 @@
   </visual>
   <collision>
-    <origin rpy="0 0 0" xyz="-0.253053 -0.228029 -0.080313"/>
+    <origin rpy="0 0 0" xyz="-0.253053 -0.228029 -0.058335"/>
     <geometry>
       <mesh filename="package://nanny_description/meshes/castor_v1_1.stl" scale="0.001 0.001 0.001"/>
@@ -359,5 +359,5 @@
   </inertial>
   <visual>
-    <origin rpy="0 0 0" xyz="-0.746563 -0.221679 -0.080313"/>
+    <origin rpy="0 0 0" xyz="-0.746563 -0.221679 -0.058335"/>
     <geometry>
       <mesh filename="package://nanny_description/meshes/castor_v1__1__1.stl" scale="0.001 0.001 0.001"/>
@@ -366,5 +366,5 @@
   </visual>
   <collision>
-    <origin rpy="0 0 0" xyz="-0.746563 -0.221679 -0.080313"/>
+    <origin rpy="0 0 0" xyz="-0.746563 -0.221679 -0.058335"/>
     <geometry>
       <mesh filename="package://nanny_description/meshes/castor_v1__1__1.stl" scale="0.001 0.001 0.001"/>
@@ -379,5 +379,5 @@
   </inertial>
   <visual>
-    <origin rpy="0 0 0" xyz="-0.354708 0.380784 -0.232713"/>
+    <origin rpy="0 0 0" xyz="-0.354708 0.380784 -0.210735"/>
     <geometry>
       <mesh filename="package://nanny_description/meshes/extrude2_1.stl" scale="0.001 0.001 0.001"/>
@@ -386,5 +386,5 @@
   </visual>
   <collision>
-    <origin rpy="0 0 0" xyz="-0.354708 0.380784 -0.232713"/>
+    <origin rpy="0 0 0" xyz="-0.354708 0.380784 -0.210735"/>
     <geometry>
       <mesh filename="package://nanny_description/meshes/extrude2_1.stl" scale="0.001 0.001 0.001"/>
@@ -399,5 +399,5 @@
   </inertial>
   <visual>
-    <origin rpy="0 0 0" xyz="-0.655908 0.372759 -0.232713"/>
+    <origin rpy="0 0 0" xyz="-0.655908 0.372759 -0.210735"/>
     <geometry>
       <mesh filename="package://nanny_description/meshes/extrude2_2.stl" scale="0.001 0.001 0.001"/>
@@ -406,5 +406,5 @@
   </visual>
   <collision>
-    <origin rpy="0 0 0" xyz="-0.655908 0.372759 -0.232713"/>
+    <origin rpy="0 0 0" xyz="-0.655908 0.372759 -0.210735"/>
     <geometry>
       <mesh filename="package://nanny_description/meshes/extrude2_2.stl" scale="0.001 0.001 0.001"/>
@@ -419,5 +419,5 @@
   </inertial>
   <visual>
-    <origin rpy="0 0 0" xyz="-0.831708 0.016584 -0.232713"/>
+    <origin rpy="0 0 0" xyz="-0.831708 0.016584 -0.210735"/>
     <geometry>
       <mesh filename="package://nanny_description/meshes/extrude2_3.stl" scale="0.001 0.001 0.001"/>
@@ -426,5 +426,5 @@
   </visual>
   <collision>
-    <origin rpy="0 0 0" xyz="-0.831708 0.016584 -0.232713"/>
+    <origin rpy="0 0 0" xyz="-0.831708 0.016584 -0.210735"/>
     <geometry>
       <mesh filename="package://nanny_description/meshes/extrude2_3.stl" scale="0.001 0.001 0.001"/>
@@ -439,5 +439,5 @@
   </inertial>
   <visual>
-    <origin rpy="0 0 0" xyz="-0.167723 0.041484 -0.232713"/>
+    <origin rpy="0 0 0" xyz="-0.167723 0.041484 -0.210735"/>
     <geometry>
       <mesh filename="package://nanny_description/meshes/extrude2_4.stl" scale="0.001 0.001 0.001"/>
@@ -446,5 +446,5 @@
   </visual>
   <collision>
-    <origin rpy="0 0 0" xyz="-0.167723 0.041484 -0.232713"/>
+    <origin rpy="0 0 0" xyz="-0.167723 0.041484 -0.210735"/>
     <geometry>
       <mesh filename="package://nanny_description/meshes/extrude2_4.stl" scale="0.001 0.001 0.001"/>
@@ -459,5 +459,5 @@
   </inertial>
   <visual>
-    <origin rpy="0 0 0" xyz="-0.346208 -0.234216 -0.232713"/>
+    <origin rpy="0 0 0" xyz="-0.346208 -0.234216 -0.210735"/>
     <geometry>
       <mesh filename="package://nanny_description/meshes/extrude2_5.stl" scale="0.001 0.001 0.001"/>
@@ -466,5 +466,5 @@
   </visual>
   <collision>
-    <origin rpy="0 0 0" xyz="-0.346208 -0.234216 -0.232713"/>
+    <origin rpy="0 0 0" xyz="-0.346208 -0.234216 -0.210735"/>
     <geometry>
       <mesh filename="package://nanny_description/meshes/extrude2_5.stl" scale="0.001 0.001 0.001"/>
@@ -479,5 +479,5 @@
   </inertial>
   <visual>
-    <origin rpy="0 0 0" xyz="-0.664208 -0.223316 -0.232713"/>
+    <origin rpy="0 0 0" xyz="-0.664208 -0.223316 -0.210735"/>
     <geometry>
       <mesh filename="package://nanny_description/meshes/extrude2_6.stl" scale="0.001 0.001 0.001"/>
@@ -486,5 +486,5 @@
   </visual>
   <collision>
-    <origin rpy="0 0 0" xyz="-0.664208 -0.223316 -0.232713"/>
+    <origin rpy="0 0 0" xyz="-0.664208 -0.223316 -0.210735"/>
     <geometry>
       <mesh filename="package://nanny_description/meshes/extrude2_6.stl" scale="0.001 0.001 0.001"/>
@@ -499,5 +499,5 @@
   </inertial>
   <visual>
-    <origin rpy="0 0 0" xyz="-0.339287 0.371159 -0.689748"/>
+    <origin rpy="0 0 0" xyz="-0.339287 0.371159 -0.66777"/>
     <geometry>
       <mesh filename="package://nanny_description/meshes/universalplate_v1__1__1.stl" scale="0.001 0.001 0.001"/>
@@ -506,5 +506,5 @@
   </visual>
   <collision>
-    <origin rpy="0 0 0" xyz="-0.339287 0.371159 -0.689748"/>
+    <origin rpy="0 0 0" xyz="-0.339287 0.371159 -0.66777"/>
     <geometry>
       <mesh filename="package://nanny_description/meshes/universalplate_v1__1__1.stl" scale="0.001 0.001 0.001"/>
@@ -519,5 +519,5 @@
   </inertial>
   <visual>
-    <origin rpy="0 0 0" xyz="-0.294756 0.377544 -0.702448"/>
+    <origin rpy="0 0 0" xyz="-0.294756 0.377544 -0.68047"/>
     <geometry>
       <mesh filename="package://nanny_description/meshes/extrude3_1.stl" scale="0.001 0.001 0.001"/>
@@ -526,5 +526,5 @@
   </visual>
   <collision>
-    <origin rpy="0 0 0" xyz="-0.294756 0.377544 -0.702448"/>
+    <origin rpy="0 0 0" xyz="-0.294756 0.377544 -0.68047"/>
     <geometry>
       <mesh filename="package://nanny_description/meshes/extrude3_1.stl" scale="0.001 0.001 0.001"/>
@@ -539,5 +539,5 @@
   </inertial>
   <visual>
-    <origin rpy="0 0 0" xyz="-0.705977 0.374254 -0.702448"/>
+    <origin rpy="0 0 0" xyz="-0.705977 0.374254 -0.68047"/>
     <geometry>
       <mesh filename="package://nanny_description/meshes/extrude3_2.stl" scale="0.001 0.001 0.001"/>
@@ -546,5 +546,5 @@
   </visual>
   <collision>
-    <origin rpy="0 0 0" xyz="-0.705977 0.374254 -0.702448"/>
+    <origin rpy="0 0 0" xyz="-0.705977 0.374254 -0.68047"/>
     <geometry>
       <mesh filename="package://nanny_description/meshes/extrude3_2.stl" scale="0.001 0.001 0.001"/>
@@ -559,5 +559,5 @@
   </inertial>
   <visual>
-    <origin rpy="0 0 0" xyz="-0.836218 0.096679 -0.702448"/>
+    <origin rpy="0 0 0" xyz="-0.836218 0.096679 -0.68047"/>
     <geometry>
       <mesh filename="package://nanny_description/meshes/extrude3_3.stl" scale="0.001 0.001 0.001"/>
@@ -566,5 +566,5 @@
   </visual>
   <collision>
-    <origin rpy="0 0 0" xyz="-0.836218 0.096679 -0.702448"/>
+    <origin rpy="0 0 0" xyz="-0.836218 0.096679 -0.68047"/>
     <geometry>
       <mesh filename="package://nanny_description/meshes/extrude3_3.stl" scale="0.001 0.001 0.001"/>
@@ -579,5 +579,5 @@
   </inertial>
   <visual>
-    <origin rpy="0 0 0" xyz="-0.718816 -0.216805 -0.702448"/>
+    <origin rpy="0 0 0" xyz="-0.718816 -0.216805 -0.68047"/>
     <geometry>
       <mesh filename="package://nanny_description/meshes/extrude3_4.stl" scale="0.001 0.001 0.001"/>
@@ -586,5 +586,5 @@
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
Commit message: commit

File: nanny_description/urdf/nanny.xacro (robot description, xacro)
@@ -806,5 +806,5 @@
   <parent link="motor_v1__1__1"/>
   <child link="wheel_v1__1__1"/>
-  <axis xyz="1.0 0.0 -0.0"/>
+  <axis xyz="1.0 0.0 0.0"/>
 </joint>
 <joint name="Rev4" type="continuous">
@@ -812,5 +812,5 @@
   <parent link="motor_v1_1"/>
   <child link="wheel_v1_1"/>
-  <axis xyz="-1.0 -0.0 -0.0"/>
+  <axis xyz="1.0 0.0 0.0"/>
 </joint>
 <joint name="Rigid8" type="fixed">
