Commit message: wokring front laser and axes are corrected

File: urdf/coach_nanny_robot.urdf (robot description, URDF)
Before this commit: robot coach_nanny_robot, 9 links, 8 joints
Links:
- removed link front_laser_link
- removed link left_caster_swivel
- removed link left_caster_wheel
- removed link rear_laser_link
- removed link right_caster_swivel
- removed link right_caster_wheel
- added link front_laser, mass 1e-5; collision mesh filename=package://nanny_description/meshes/front_laser.STL; visual mesh filename=package://nanny_description/meshes/front_laser.STL
- added link left_caster, mass 0.470013684691794; collision mesh filename=package://nanny_description/meshes/left_caster.STL; visual mesh filename=package://nanny_description/meshes/left_caster.STL
- added link left_swivel, mass 1.62791183303881; collision mesh filename=package://nanny_description/meshes/left_swivel.STL; visual mesh filename=package://nanny_description/meshes/left_swivel.STL
- added link rear_laser, mass 1e-5; collision mesh filename=package://nanny_description/meshes/rear_laser.STL; visual mesh filename=package://nanny_description/meshes/rear_laser.STL
- added link right_caster, mass 0.470013684691794; collision mesh filename=package://nanny_description/meshes/right_caster.STL; visual mesh filename=package://nanny_description/meshes/right_caster.STL
- added link right_swivel, mass 1.62791183303881; collision mesh filename=package://nanny_description/meshes/right_swivel.STL; visual mesh filename=package://nanny_description/meshes/right_swivel.STL
- link base_link: mass 26.8043249525411 -> 26.1616258468403
- link left_wheel: mass 0.84408 -> 0.844079114777031
- link right_wheel: mass 0.84408 -> 0.844079114777032
Joints:
- removed joint base_link_left_caster_swivel
- removed joint base_link_right_caster_swivel
- removed joint left_caster_swivel_left_caster_wheel
- removed joint right_caster_swivel_right_caster_wheel
- added joint base_link_left_swivel: type continuous, parent base_link, child left_swivel, origin xyz=-0.1984 0.1964315 0.0925375 rpy=0 0 0, axis 0 0 1
- added joint base_link_right_swivel: type continuous, parent base_link, child right_swivel, origin xyz=-0.1984 -0.1964315 0.0925375 rpy=0 0 0, axis 0 0 1
- added joint left_swivel_left_caster: type continuous, parent left_swivel, child left_caster, origin xyz=-0.04445 -0.000507999999999981 -0.0714375 rpy=0 0 0, axis 0 -1 0
- added joint right_swivel_right_caster: type continuous, parent right_swivel, child right_caster, origin xyz=-0.04445 -0.000508000000000036 -0.0714375 rpy=0 0 0, axis 0 1 0
- joint base_link_front_laser: axis 0 0 0 -> 0 0 1; child front_laser_link -> front_laser; limit (none) -> lower=0 upper=0 effort=0 velocity=0; origin xyz=0 0 0 rpy=0 0 0 -> xyz=0.26865 0 0.043175 rpy=0 0 0; type fixed -> revolute
- joint base_link_left_wheel: axis 1 0 0 -> 0 1 0; origin xyz=0.27871 -0.17336 0.048701 rpy=0 0 0 -> xyz=0.173356333637394 0.27870625 0.0487011859215695 rpy=0 0 0
- joint base_link_rear_laser: axis 0 0 0 -> 0 0 1; child rear_laser_link -> rear_laser; limit (none) -> lower=0 upper=0 effort=0 velocity=0; origin xyz=0 0 0 rpy=0 0 0 -> xyz=-0.27182 0 0.043175 rpy=0 0 0; type fixed -> revolute
- joint base_link_right_wheel: axis 1 0 0 -> 0 1 0; origin xyz=-0.27871 -0.17336 0.048701 rpy=0 0 0 -> xyz=0.17336 -0.27871 0.048701 rpy=0 0 0
