Commit message: update urdf

File: urdf/covid_killer_robot.urdf (robot description, URDF)
Before this commit: robot covid_killer_robot, 12 links, 11 joints
Links:
- link base_link: mass 32.099 -> 44.766149285195
Joints:
- joint base_link_back_left_swivel: origin xyz=0.254 0.254 0.092538 rpy=0 0 -1.5708 -> xyz=-0.254 0.254 0.092538 rpy=0 0 0
- joint base_link_back_right_swivel: origin xyz=-0.254 0.254 0.092538 rpy=0 0 -1.5708 -> xyz=-0.254 -0.254 0.092538 rpy=0 0 0
- joint base_link_front_laser: axis 0 0 -1 -> 0 0 1; origin xyz=0 -0.38239 0.15967 rpy=0 0 -1.5708 -> xyz=0.38239 0 0.15967 rpy=0 0 0; type revolute -> fixed
- joint base_link_front_left_swivel: origin xyz=0.254 -0.254 0.092538 rpy=0 0 -1.5708 -> xyz=0.254 0.254 0.092538 rpy=0 0 0
- joint base_link_front_right_swivel: origin xyz=-0.254 -0.254 0.092538 rpy=0 0 -1.5708 -> xyz=0.254 -0.254 0.092538 rpy=0 0 0
- joint base_link_left_wheel: limit (none) -> effort=10000 velocity=1000; origin xyz=0.28302 0 0.048701 rpy=0 0 -1.5708 -> xyz=0 0.28302 0.048701 rpy=0 0 0
- joint base_link_right_wheel: limit (none) -> effort=10000 velocity=1000; origin xyz=-0.28302 0 0.048701 rpy=0 0 -1.5708 -> xyz=0 -0.28302 0.048701 rpy=0 0 0

Commit message: Changed frame name to 'front_laser' from 'odom'

File: urdf/covid_killer_robot.urdf (robot description, URDF)
Before this commit: robot covid_killer_robot, 12 links, 11 joints
Joints:
- joint base_link_left_wheel: limit effort=10000 velocity=1000 -> (none)
- joint base_link_right_wheel: limit effort=10000 velocity=1000 -> (none)

Commit message: added cameras and lidar

File: urdf/covid_killer_robot.urdf (robot description, URDF)
Before this commit: robot covid_killer_robot, 12 links, 11 joints
Links:
- added link front_camera, mass 0.1; collision box size=0.05 0.05 0.05; visual box size=0.05 0.05 0.05
- added link rear_camera, mass 0.1; collision box size=0.05 0.05 0.05; visual box size=0.05 0.05 0.05
- added link rear_laser, mass 0.36783; collision mesh filename=package://nanny_description/meshes/front_laser.STL; visual mesh filename=package://nanny_description/meshes/front_laser.STL
Joints:
- added joint base_link_front_camera: type fixed, parent base_link, child front_camera, origin xyz=0.38239 0 0.25 rpy=0 0 0, axis 0 1 0
- added joint base_link_rear_camera: type fixed, parent base_link, child rear_camera, origin xyz=-0.38239 0 0.25 rpy=0 0 3.14159, axis 0 1 0
- added joint base_link_rear_laser: type revolute, parent base_link, child rear_laser, origin xyz=-0.38239 0 0.15967 rpy=0 0 3.14159, axis 0 0 -1, limit lower=0 upper=0 effort=0 velocity=0
